File: KiCad/BT/BT.kicad_pcb (KiCad board)
At the start: 4 copper layers, 13.8 x 31.5 mm, 54 parts, among them J1 UJC-HP-3-SMT-TR, J2 2328702-8, J3 Conn_01x05, SW1 Val**, U1 QFN40P120X130X45-6N, U2 SON95P300X300X100-7N-D, U3 STM6601CQ2BDM6F, U4 BMD-350-A-R, U5 UDFN6, U6 UDFN6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

Commit message: minor updates
Parts:
- moved R10 0.05 mm to (107.5, 59.4)
- moved R20 0.05 mm to (107.5, 60.5)
- moved R3 0.05 mm to (107.5, 61.6)
- moved R4 0.05 mm to (107.5, 62.7)
- moved R9 0.05 mm to (107.5, 58.3)
Routing:
- net XSHUT2: track 24.6 -> 24.0 mm
- net GND: track 40.7 -> 40.2 mm, vias 69 -> 67

Commit message: updated
Parts:
- moved R13 0.06 mm to (107.5, 69.3)
- moved R16 0.06 mm to (107.5, 67.1)
- moved R22 0.06 mm to (107.5, 70.4)
- moved R24 0.06 mm to (107.5, 64.9)
- moved R25 0.06 mm to (107.5, 68.2)
- moved R26 0.06 mm to (107.5, 66.0)
Routing:
- net GND: track 40.2 -> 40.1 mm, vias 67 -> 70
Other:
- board text added: "BT_v6.1"
- board text removed: "BT_v6.0"

Commit message: swapped SWDIO/SWCLK, BM pin moved to AN4
Parts:
- SW1: value Val** -> PTS840ESDPMSMTRLFS
- U1: value QFN40P120X130X45-6N -> LDK130PU-R
- U2: value SON95P300X300X100-7N-D -> STBC08PMR
- U5, U6, U7: value UDFN6 -> SSM6L61NU
- Y1: value ECS-.327-7-34R-TR -> ECS-.327-CDX-2216
Connections:
- J3 pad 3: SWDCLK -> SWDIO
- J3 pad 4: SWDIO -> SWDCLK
- U4 pad 32: LED_EN -> BM_EN
- U4 pad 4: SWDIO -> SWDCLK
- U4 pad 45: BM_EN -> BM
- U4 pad 5: SWDCLK -> SWDIO
Routing:
- net BM: track 16.3 -> 21.2 mm
- net XSHUT1: track 24.2 -> 22.5 mm
- net PS_HOLD: track 9.16 -> 8.45 mm
- net GND: track 40.1 -> 39.5 mm
Other:
- board text added: "BT_v7.0"
- board text removed: "BT_v6.1"
